Commit message: Created mesh based URDF, issue #5

File: packages/robot_viz/urdf/simple_robot.urdf (robot description, URDF)
Before this commit: robot simple_robot, 2 links, 1 joints
Links:
- link base_link: geometry visual cylinder length=0.75 radius=0.5
- link link1: geometry visual mesh filename=package://robot_viz/urdf/meshes/link1_body.stl scale=0.001 0.001 0.001
