Commit message: Finished solving and documenting issue #5

File: packages/robot_viz/urdf/robot_builder.urdf (robot description, URDF)
Before this commit: robot robot_v1, 3 links, 2 joints
Links:
- added link link3, mass 0.0; collision box size=1 0.2 0.2; visual mesh filename=package://robot_viz/urdf/meshes/link1_body.stl scale=0.001 0.001 0.001
Joints:
- added joint joint_link2_link3: type revolute, parent link2, child link3, origin xyz=1.0 0.0 0 rpy=0.0 0.0 1.57079632679, axis 0.0 0.0 1.0, limit lower=-3.14159265359 upper=6.28318530718 effort=10 velocity=10
- joint joint_base_link_link1: limit lower=0 upper=6.28318530718 effort=10 velocity=10 -> lower=-3.14159265359 upper=3.14159265359 effort=10 velocity=10
- joint joint_link1_link2: limit lower=0 upper=6.28318530718 effort=10 velocity=10 -> lower=-3.14159265359 upper=3.14159265359 effort=10 velocity=10; origin xyz=1.0 0.0 0 rpy=0.0 -1.57079632679 0.0 -> xyz=0.0 0.0 0 rpy=0.0 -1.57079632679 0.0

File: packages/robot_viz/urdf/robot_builder.xacro (robot description, xacro)
@@ -17,5 +17,5 @@
     <!-- parent: Parent link name [default is "base_link"] -->
     <!-- child: Name of the child link (required) -->
-    <!-- file_path: Path to the mesh file (stl or dae) for the link -->
+    <!-- file_path: Path to the mesh file (stl or dae) for the child link -->
     <!-- mesh_scale: Scaling factor of the mesh that is imported [default is 0.001] -->
     <!-- min_q: Minimum actuation value of the revolute joint -->
@@ -67,4 +67,5 @@
                 <inertia ixx="0.0" ixy="0.0" ixz="0.0" iyy="0.0" iyz="0.0" izz="0.0"/>
             </inertial>
+            <!-- Visual properties here -->
             <visual>
                 <origin xyz="0.0 0.0 0.0" rpy="0.0 0.0 0.0"/>
@@ -76,4 +77,5 @@
                 </material>
             </visual>
+            <!-- Collision properties here -->
             <collision>
                 <origin xyz="0.0 0.0 0.0" rpy="0.0 0.0 0.0"/>
@@ -86,6 +88,19 @@
     <!-- Child links -->
     <!-- Link 1 -->
-    <xacro:attach_link parent="base_link" child="link1" file_path="${link1_mesh}" min_q="0" max_q="${2 * pi}">
+    <xacro:attach_link parent="base_link" child="link1" file_path="${link1_mesh}" min_q="${-pi}" max_q="${pi}">
+        <!-- Origin of child frame in parent frame -->
         <origin xyz="0.0 0.0 0.15" rpy="0.0 0.0 0.0"/>
+        <!-- Collision boundary -->
+        <box size="1 0.2 0.2"/>
+        <!-- Inertial properties of the link -->
+        <inertia_block>
+            <origin xyz="0.0 0.0 0.0" rpy="0.0 0.0 0.0"/>
+            <mass value="0.0"/>
+            <inertia ixx="0.0" ixy="0.0" ixz="0.0" iyy="0.0" iyz="0.0" izz="0.0"/>
+        </inertia_block>
+    </xacro:attach_link>
+    <!-- Link 2 -->
+    <xacro:attach_link parent="link1" child="link2" file_path="${link1_mesh}" min_q="${-pi}" max_q="${pi}">
+        <origin xyz="0.0 0.0 0" rpy="0.0 ${-pi / 2} 0.0"/>
         <box size="1 0.2 0.2"/>
         <inertia_block>
@@ -95,14 +110,3 @@
         </inertia_block>
     </xacro:attach_link>
-    <!-- Link 2 -->
-    <xacro:attach_link parent="link1" child="link2" file_path="${link1_mesh}" min_q="0" max_q="${2 * pi}">
-        <origin xyz="1.0 0.0 0" rpy="0.0 ${-pi / 2} 0.0"/>
-        <box size="1 0.2 0.2"/>
-        <inertia_block>
-            <origin xyz="0.0 0.0 0.0" rpy="0.0 0.0 0.0"/>
-            <mass value="0.0"/>
-            <inertia ixx="0.0" ixy="0.0" ixz="0.0" iyy="0.0" iyz="0.0" izz="0.0"/>
-        </inertia_block>
-    </xacro:attach_link>
-    <!-- "xacro --check-order robot_builder.xacro -o robot_builder.urdf" for running -->
 </robot>
